Commit message: some odometry improvements

File: nano_atrv_description/urdf/nano_atrv.urdf (robot description, URDF)
Before this commit: robot nano_atrv, 4 links, 3 joints
Links:
- added link left_steer_link
- added link left_wheel
- added link left_wheel_link
- added link rear_steer_link
- added link rear_wheel_link
- added link right_steer_link
- added link right_wheel
- added link right_wheel_link
Joints:
- added joint base_link_to_left_steer: type fixed, parent base_link, child left_steer_link, origin xyz=0.175 0.1775 -0.1 rpy=0 0 0
- added joint base_link_to_rear_steer: type fixed, parent base_link, child rear_steer_link, origin xyz=-0.175 0 -0.1 rpy=0 0 0
- added joint base_link_to_right_steer: type fixed, parent base_link, child right_steer_link, origin xyz=0.175 -0.1775 -0.1 rpy=0 0 0
- added joint left_steer_joint: type revolute, parent left_steer_link, child left_wheel_link, origin xyz=0 0 0 rpy=0 0 0, axis 0 0 1, limit lower=-1.57 upper=1.57 effort=10 velocity=2
- added joint left_wheel_joint: type continuous, parent left_wheel_link, child left_wheel, origin xyz=0 0.08 0 rpy=0 0 1.5708, axis -1 0 0
- added joint rear_steer_joint: type revolute, parent rear_steer_link, child rear_wheel_link, origin xyz=0 0 0 rpy=0 0 0, axis 0 0 1, limit lower=-3.1415 upper=3.1415 effort=10 velocity=2
- added joint right_steer_joint: type revolute, parent right_steer_link, child right_wheel_link, origin xyz=0 0 0 rpy=0 0 0, axis 0 0 1, limit lower=-1.57 upper=1.57 effort=10 velocity=2
- added joint right_wheel_joint: type continuous, parent right_wheel_link, child right_wheel, origin xyz=0 -0.08 0 rpy=0 0 -1.5708, axis 1 0 0

Commit message: inverse kinetmatics, arm control

File: nano_atrv_description/urdf/nano_atrv.urdf (robot description, URDF)
Before this commit: robot nano_atrv, 12 links, 11 joints
Links:
- added link base_link_arm
Joints:
- added joint base_link_to_arm: type fixed, parent base_link, child base_link_arm, origin xyz=0.145 0 0 rpy=0 0 0

Commit message: camera tilt

File: nano_atrv_description/urdf/nano_atrv.urdf (robot description, URDF)
Before this commit: robot nano_atrv, 13 links, 12 joints
Joints:
- joint base_link_to_camera_link: origin xyz=0.07 0 0.35 rpy=0 0 0 -> xyz=0.08 0 0.34 rpy=0 0.523 0

Commit message: nav2 test config

File: nano_atrv_description/urdf/nano_atrv.urdf (robot description, URDF)
Before this commit: robot nano_atrv, 13 links, 12 joints
Joints:
- joint base_link_to_camera_link: origin xyz=0.08 0 0.34 rpy=0 0.523 0 -> xyz=0.08 0 0.39 rpy=0 0.523 0

Commit message: docs update, arm stow

File: nano_atrv_description/urdf/nano_atrv.urdf (robot description, URDF)
Before this commit: robot nano_atrv, 13 links, 12 joints
Joints:
- joint base_link_to_camera_link: origin xyz=0.08 0 0.39 rpy=0 0.523 0 -> xyz=0.08 0.05 0.28 rpy=0 0.8726 0

Commit message: 3D printed part meshes, urdf fix

File: nano_atrv_description/urdf/nano_atrv.urdf (robot description, URDF)
Before this commit: robot nano_atrv, 13 links, 12 joints
Joints:
- joint base_link_to_camera_link: origin xyz=0.08 0.05 0.28 rpy=0 0.8726 0 -> xyz=0.08 0.05 0.285 rpy=0 0.8029 0
- joint base_link_to_laser: origin xyz=0 0 0.3 rpy=0 3.1415 0 -> xyz=0 0 0.23 rpy=0 3.1415 0
